Commit message: p1: harden the `stuck` claim with six more rollouts, and fix what that exposed
The previous result rested on one `stuck` rollout, so its seven frames were one
robot in one pose imaged seven times. Six more rollouts vary the obstacle:
oblique wall, dim wall, V-funnel, wall edge, a slot narrower than the robot, and
a kerb too low for the camera to see. All seven run an identical drive script so
the scene is the only variable.

The claim survives, much larger: 9 rollouts, 103 labelled frames, 206
evaluations, 0 errors, 100% parse coverage. llava-phi3 names `stuck` once in 110
attempts (0/55 visual, 1/55 grounded) and scores below the always-guess baseline
in all four configurations. From the image alone it never once answers
`failed: true`. 71% of grounded answers set `failed: false` while naming a
failure mode.

Two things the new data exposed, both of which changed the harness:

- Different stall scenes render the *same picture*. At contact the camera is
  ~5 cm out and its 60 deg FOV spans ~6 cm, so any larger obstacle fills the
  frame and approach angle, shape and lighting are invisible. The four
  wall-type rollouts produced 30 byte-identical frames. Keyframes now carry a
  `pixel_sha1`, extraction reports how many are pixel-unique, and scoring prints
  a duplicate-weighted accuracy with a matching weighted baseline. 103 frames
  are 51 images; the 55 `stuck` frames are 15.

- The oscillation labeller was wrong. Its extent cap also fires on a *straight*
  run shorter than ~0.8 m, because a straight line's extent is half its path;
  every earlier scenario travelled further and hid it. Replaced with a
  path/extent shape test (real oscillation 6.6-12.0, straight lines 1.2-2.3).
  The three pre-existing runs re-label byte-for-byte identically, so the
  previously published numbers were unaffected.

Worlds now share tb3_base.xacro; tb3_wall expands semantically identically to
the version it replaces. verify_readme_numbers.py re-derives all 29 numbers the
p1 README quotes straight from the data.

File: harness/recorder/worlds/tb3_wall.sdf.xacro (robot description, xacro)
@@ -1,111 +1,16 @@
 <?xml version="1.0"?>
+<!--
+  tb3_sandbox plus one flat slab across the lane.
+  A robot spawned at (-2.0, -0.5) facing +x meets it head-on after about 1 m.
+  This is the original `stuck` scene; `tb3_corner`, `tb3_gap` and `tb3_wall_dim`
+  vary the obstacle around it so the class rests on more than one situation.
+-->
 <sdf version="1.6" xmlns:xacro="http://www.ros.org/wiki/xacro">
   <xacro:arg name="headless" default="true"/>
+  <!-- relative includes resolve against this file's directory, not the cwd -->
+  <xacro:include filename="tb3_base.xacro"/>
   <world name="default">
-    <plugin
-      filename="gz-sim-physics-system"
-      name="gz::sim::systems::Physics">
-    </plugin>
-    <plugin
-      filename="gz-sim-user-commands-system"
-      name="gz::sim::systems::UserCommands">
-    </plugin>
-  <xacro:unless value="$(arg headless)">
-    <plugin
-      filename="gz-sim-scene-broadcaster-system"
-      name="gz::sim::systems::SceneBroadcaster">
-    </plugin>
-  </xacro:unless>
-    <plugin
-      filename="gz-sim-sensors-system"
-      name="gz::sim::systems::Sensors">
-      <render_engine>ogre2</render_engine>
-    </plugin>
-    <plugin
-      filename="gz-sim-imu-system"
-      name="gz::sim::systems::Imu">
-    </plugin>
-    <light name='sun' type='directional'>
-        <cast_shadows>0</cast_shadows>
-        <pose>0 0 10 0 0 0</pose>
-        <diffuse>0.8 0.8 0.8 1</diffuse>
-        <specular>0.8 0.8 0.8 1</specular>
-        <attenuation>
-            <range>1000</range>
-            <constant>0.9</constant>
-            <linear>0.01</linear>
-            <quadratic>0.001</quadratic>
-        </attenuation>
-        <direction>-0.5 0.1 -0.9</direction>
-    </light>
-    <model name='ground_plane'>
-        <static>1</static>
-        <link name='link'>
-            <collision name='collision'>
-                <geometry>
-                    <plane>
-                        <normal>0 0 1</normal>
-                        <size>100 100</size>
-                    </plane>
-                </geometry>
-                <max_contacts>10</max_contacts>
-            </collision>
-            <visual name='visual'>
-                <geometry>
-                    <plane>
-                        <normal>0 0 1</normal>
-                        <size>100 100</size>
-                    </plane>
-                </geometry>
-                <material>
-                    <ambient>0.8 0.8 0.8 1</ambient>
-                    <diffuse>0.8 0.8 0.8 1</diffuse>
-                    <specular>0.8 0.8 0.8 1</specular>
-                </material>
-            </visual>
-        </link>
-    </model>
-    <scene>
-      <shadows>0</shadows>
-    </scene>
-    <physics name='3ms' type='ode'>
-        <max_step_size>0.003</max_step_size>
-        <real_time_factor>1</real_time_factor>
-    </physics>
-    <model name="turtlebot3_world">
-      <static>1</static>
-      <include>
-        <uri>model://turtlebot3_world</uri>
-      </include>
-    </model>
-    <!-- ADDED (this world is tb3_sandbox plus the wall below).
-         The stock sandbox is nine cylinders in a 3x3 grid at
-         (x,y) in {-1.1, 0, 1.1}^2. A robot driven at them glances off the
-         curved surface and scrubs sideways instead of wedging: the `stuck_wall`
-         scenario ended 7.8 m along a deflected path at yaw 143 deg, never once
-         tripping the stall test. Round obstacles cannot produce a reliable stall.
-         This is a flat slab across the lane at y = -0.5, which a robot spawned
-         at (-2.0, -0.5) facing +x meets head-on after ~1 m. Flat and static, so
-         contact is a genuine stall rather than a deflection. -->
-    <model name="stall_wall">
-      <static>true</static>
-      <pose>-0.85 -0.5 0.25 0 0 0</pose>
-      <link name="link">
-        <collision name="collision">
-          <geometry>
-            <box><size>0.15 1.4 0.5</size></box>
-          </geometry>
-        </collision>
-        <visual name="visual">
-          <geometry>
-            <box><size>0.15 1.4 0.5</size></box>
-          </geometry>
-          <material>
-            <ambient>0.75 0.25 0.2 1</ambient>
-            <diffuse>0.75 0.25 0.2 1</diffuse>
-          </material>
-        </visual>
-      </link>
-    </model>
+    <xacro:tb3_base_world headless="$(arg headless)"/>
+    <xacro:slab name="stall_wall" x="-0.85" y="-0.5"/>
   </world>
 </sdf>
