Commit message: Phase 2: language-queryable semantic SLAM, and where it stops working
slam_toolbox builds the metric map; llava-phi3 labels keyframes; each label is
anchored to the pose it was seen from, so "where did you last see the chair?"
returns a coordinate the robot then drives to.

Half of it works. Over one 12.27 m circuit the SLAM pose error is 8 mm median
and the labels are clean (26/26 correct on empty frames), placing the chair to
0.08 m and the bookshelf to 0.22 m against a 2.50 m trivial baseline. The sofa
lands at 1.46 m and the table is never located.

The failing half is the finding: a whole-image label names what is there but
not where. Taking the camera axis as the bearing is wrong by 23 deg median, so
triangulation loses to naive averaging. Asking the model which third of the
frame the object occupies made it worse -- it answered `left` on 9 of 10 frames
and `centre` on none, injecting a systematic offset. The number that predicts
localisation error is the signed bearing bias, not the absolute one.

Also recorded: Nav2's full stack does not run on this machine (15 processes,
load average 21 on 4 cores, robot never moved), so the demo uses slam_toolbox
alone plus a turn-then-go controller in drive.py --mode goto.

verify_readme_numbers.py re-derives all 29 numbers the README quotes.

File: harness/recorder/worlds/tb3_base.xacro (robot description, xacro)
@@ -21,5 +21,13 @@
 -->
 <robot xmlns:xacro="http://www.ros.org/wiki/xacro">
-  <xacro:macro name="tb3_base_world" params="headless light_diffuse:='0.8 0.8 0.8 1'">
+  <!--
+    `scenery` controls the stock turtlebot3_world (hexagon wall + nine cylinders).
+    p1 wants it: those cylinders are what a robot deflects off, and they are the
+    reason the flat slab had to be added. p2 does not: it needs a room with
+    *nameable* objects in it, and nine untextured cylinders are exactly the
+    flat-shaded geometry p1 measured small VLMs failing on.
+  -->
+  <xacro:macro name="tb3_base_world"
+               params="headless light_diffuse:='0.8 0.8 0.8 1' scenery:='true'">
     <plugin
       filename="gz-sim-physics-system"
@@ -92,4 +100,5 @@
         <real_time_factor>1</real_time_factor>
     </physics>
+    <xacro:if value="${scenery}">
     <model name="turtlebot3_world">
       <static>1</static>
@@ -98,4 +107,5 @@
       </include>
     </model>
+    </xacro:if>
   </xacro:macro>
   <!--
